File: PCB/microkey.kicad_pcb (KiCad board)
At the start: 2 copper layers, 35 x 17 mm, 43 parts, among them J1 Button, U1 RP2350_60QFN, U2 TPS7A2033PDBVR, Y1 ABM8-272-T3

Commit message: readme and bom
Parts:
- moved R8 0.41 mm to (210.0, 106.8)
- moved R7 0.40 mm to (210.0, 107.8)
- moved U3 0.35 mm to (209.8, 111.0)
Routing:
- net +3V3: track 73.6 -> 74.4 mm
- net /USB_D+: track 7.06 -> 6.53 mm
- net /USB_D-: track 6.83 -> 6.32 mm
- net GND: track 71.7 -> 71.2 mm, vias 20 -> 21
Other:
- board text added: "µ"

Commit message: edge plating!!
Parts:
- moved C1 27.9 mm to (188.5, 103.7), turned to -135 degrees
- moved R4 14.3 mm to (195.8, 113.8)
- moved TP1 13.7 mm to (193.2, 113.2)
- moved C5 13.4 mm to (213.0, 111.5)
- moved R5 2.54 mm to (207.0, 101.5)
- moved U2 0.97 mm to (212.1, 102.4)
- moved TP4 0.76 mm to (200.0, 113.0)
- moved TP3 0.73 mm to (198.0, 113.0)
- moved C15 0.56 mm to (202.3, 101.2)
- moved C14 0.53 mm to (213.8, 109.5)
- moved R16 0.49 mm to (214.1, 103.5)
- moved C13 0.35 mm to (195.8, 112.5), turned to 180 degrees
- moved R6 0.17 mm to (206.0, 113.6)
Routing:
- net GND: track 71.2 -> 66.3 mm, vias 21 -> 19
- net +3V3: track 74.4 -> 72.7 mm
- net VBUS: track 44.0 -> 42.5 mm
- net Net-(R4-Pad1): track 3.66 -> 2.20 mm
- net /VREG_AVDD: track 7.04 -> 8.37 mm
Other:
- board text added: "3mm"
- board text added: "A"
- board text added: "C"
- board text added: "Please edge plate all sides (circled) except the C area. If needed, please use A and B for edge tabs. Please try to keep A and B edge plated if possible."
